Commit message: feat: simulation; admittance is working

File: polymetis/polymetis/data/franka_panda/panda_arm_hand.urdf (robot description, URDF)
Before this commit: robot panda, 12 links, 11 joints
Links:
- link panda_hand: mass None -> 0.73
- link panda_leftfinger: mass None -> 0.015
- link panda_link0: mass None -> 0.629769
- link panda_rightfinger: mass None -> 0.015

Commit message: fix: admittance controller is ready

File: polymetis/polymetis/data/franka_panda/panda_arm_hand.urdf (robot description, URDF)
Before this commit: robot panda, 12 links, 11 joints
Joints:
- joint panda_finger_joint1: axis 0 1 0 -> (none); limit lower=-0.001 upper=0.04 effort=20 velocity=0.3 -> (none); type prismatic -> fixed
- joint panda_finger_joint2: axis 0 -1 0 -> (none); limit lower=-0.001 upper=0.04 effort=20 velocity=0.3 -> (none); type prismatic -> fixed
